Commit message: add my ground plane and poll and ball :

File: onigiri_war/models/hoge.gazebo.xacro (robot description, xacro)
@@ -17,7 +17,5 @@
   </gazebo>
   <gazebo reference="wheel_right_link">
-    <mu1>0.1</mu1>
-    <mu2>0.1</mu2>
-    <kp>500000.0</kp>
+    <mu1>0.1</mu1> <mu2>0.1</mu2> <kp>500000.0</kp>
     <kd>10.0</kd>
     <minDepth>0.001</minDepth>
@@ -157,6 +155,11 @@
           <distortionT1>0.0</distortionT1>
           <distortionT2>0.0</distortionT2>
-        </plugin>
-      </sensor>
+        </plugin> </sensor>
     </gazebo>
+  <gazebo reference="ball">
+    <material>Gazebo/Red</material>
+  </gazebo>
+  <gazebo reference="poll">
+    <material>Gazebo/DarkGrey</material>
+  </gazebo>
 </robot>

File: onigiri_war/models/hoge.urdf.xacro (robot description, xacro)
@@ -215,3 +215,27 @@
     </visual>
   </link>
+  <joint name="poll_joint" type="fixed">
+    <origin rpy="0 0 0" xyz="-0.09 0.0 0.17"/>
+    <parent link="base_link"/>
+    <child link="poll"/>
+  </joint>
+  <link name="poll">
+    <visual>
+      <geometry>
+        <cylinder length="0.05" radius="0.002"/>
+      </geometry>
+    </visual>
+  </link>
+  <joint name="ball_joint" type="fixed">
+    <origin rpy="0 0 0" xyz="-0.09 0.0 0.21"/>
+    <parent link="base_link"/>
+    <child link="ball"/>
+  </joint>
+  <link name="ball">
+    <visual>
+      <geometry>
+        <sphere radius="0.025"/>
+      </geometry>
+    </visual>
+  </link>
 </robot>
