Commit message: add marker to robot

File: onigiri_war/models/hoge.urdf.xacro (robot description, xacro)
@@ -142,3 +142,76 @@
     </visual>
   </link>
+ <!--One Night ROBOCON add-->
+  <joint name="tag1_joint" type="fixed">
+    <origin rpy="-1.571 3.1415 0" xyz="-0.03 0.07 0.09"/>
+    <parent link="base_link"/>
+    <child link="tag1"/>
+  </joint>
+  <link name="tag1">
+    <visual>
+      <geometry>
+          <mesh filename="package://onigiri_war/models/tags/0050g.dae" scale="1.0 1.0 1.0" />
+      </geometry>
+    </visual>
+  </link>
+  <joint name="tag1-1_joint" type="fixed">
+    <origin rpy="-1.571 3.1415 0" xyz="-0.03 0.069 0.09"/>
+    <parent link="base_link"/>
+    <child link="tag1-1"/>
+  </joint>
+  <link name="tag1-1">
+    <visual>
+      <geometry>
+          <mesh filename="package://onigiri_war/models/tags/test.dae" scale="1.0 1.0 1.0"/>
+      </geometry>
+    </visual>
+  </link>
+  <joint name="tag2_joint" type="fixed">
+    <origin rpy="1.571 0 0" xyz="-0.03 -0.07 0.09"/>
+    <parent link="base_link"/>
+    <child link="tag2"/>
+  </joint>
+  <link name="tag2">
+    <visual>
+      <geometry>
+          <mesh filename="package://onigiri_war/models/tags/0051g.dae" scale="1.0 1.0 1.0" />
+      </geometry>
+    </visual>
+  </link>
+  <joint name="tag2-1_joint" type="fixed">
+    <origin rpy="1.571 0 0" xyz="-0.03 -0.069 0.09"/>
+    <parent link="base_link"/>
+    <child link="tag2-1"/>
+  </joint>
+  <link name="tag2-1">
+    <visual>
+      <geometry>
+          <mesh filename="package://onigiri_war/models/tags/test.dae" scale="1.0 1.0 1.0"/>
+      </geometry>
+    </visual>
+  </link>
+  <joint name="tag3_joint" type="fixed">
+    <origin rpy="1.571 0 -1.571" xyz="-0.101 0.0 0.09"/>
+    <parent link="base_link"/>
+    <child link="tag3"/>
+  </joint>
+  <link name="tag3">
+    <visual>
+      <geometry>
+          <mesh filename="package://onigiri_war/models/tags/0052g.dae" scale="1.0 1.0 1.0" />
+      </geometry>
+    </visual>
+  </link>
+  <joint name="tag3-1_joint" type="fixed">
+    <origin rpy="1.571 0 -1.571" xyz="-0.10 0.0 0.09"/>
+    <parent link="base_link"/>
+    <child link="tag3-1"/>
+  </joint>
+  <link name="tag3-1">
+    <visual>
+      <geometry>
+          <mesh filename="package://onigiri_war/models/tags/test.dae" scale="1.0 1.0 1.0"/>
+      </geometry>
+    </visual>
+  </link>
 </robot>

Commit message: modify field ground and tag size

File: onigiri_war/models/hoge.urdf.xacro (robot description, xacro)
@@ -151,5 +151,6 @@
     <visual>
       <geometry>
-          <mesh filename="package://onigiri_war/models/tags/0050g.dae" scale="1.0 1.0 1.0" />
+          <!-- 120mm x 0.666 = 80mm -->
+          <mesh filename="package://onigiri_war/models/tags/0050g.dae" scale="0.666 0.666 1.0" />
       </geometry>
     </visual>
@@ -163,5 +164,5 @@
     <visual>
       <geometry>
-          <mesh filename="package://onigiri_war/models/tags/test.dae" scale="1.0 1.0 1.0"/>
+          <mesh filename="package://onigiri_war/models/tags/test.dae" scale="0.666 0.666 1.0"/>
       </geometry>
     </visual>
@@ -175,5 +176,5 @@
     <visual>
       <geometry>
-          <mesh filename="package://onigiri_war/models/tags/0051g.dae" scale="1.0 1.0 1.0" />
+          <mesh filename="package://onigiri_war/models/tags/0051g.dae" scale="0.666 0.666 1.0" />
       </geometry>
     </visual>
@@ -187,5 +188,5 @@
     <visual>
       <geometry>
-          <mesh filename="package://onigiri_war/models/tags/test.dae" scale="1.0 1.0 1.0"/>
+          <mesh filename="package://onigiri_war/models/tags/test.dae" scale="0.666 0.666 1.0"/>
       </geometry>
     </visual>
@@ -199,5 +200,5 @@
     <visual>
       <geometry>
-          <mesh filename="package://onigiri_war/models/tags/0052g.dae" scale="1.0 1.0 1.0" />
+          <mesh filename="package://onigiri_war/models/tags/0052g.dae" scale="0.666 0.666 1.0" />
       </geometry>
     </visual>
@@ -211,10 +212,10 @@
     <visual>
       <geometry>
-          <mesh filename="package://onigiri_war/models/tags/test.dae" scale="1.0 1.0 1.0"/>
+          <mesh filename="package://onigiri_war/models/tags/test.dae" scale="0.666 0.666 1.0"/>
       </geometry>
     </visual>
   </link>
   <joint name="poll_joint" type="fixed">
-    <origin rpy="0 0 0" xyz="-0.09 0.0 0.17"/>
+    <origin rpy="0 0 0" xyz="-0.09 0.0 0.12"/>
     <parent link="base_link"/>
     <child link="poll"/>
