Commit message: modify field size etc

File: burger_war/models/hoge.urdf.xacro (robot description, xacro)
@@ -3,5 +3,5 @@
   <xacro:include filename="$(find turtlebot3_description)/urdf/common_properties.xacro"/>
   <!-- xacro:include filename="$(find turtlebot3_description)/urdf/turtlebot3_burger.gazebo.xacro"/-->
-  <xacro:include filename="$(find onigiri_war)/models/hoge.gazebo.xacro"/>
+  <xacro:include filename="$(find burger_war)/models/hoge.gazebo.xacro"/>
   <link name="base_footprint"/>
   <joint name="base_joint" type="fixed">
@@ -152,5 +152,5 @@
       <geometry>
           <!-- 120mm x 0.666 = 80mm -->
-          <mesh filename="package://onigiri_war/models/tags/0050g.dae" scale="0.666 0.666 1.0" />
+          <mesh filename="package://burger_war/models/tags/0050g.dae" scale="0.666 0.666 1.0" />
       </geometry>
     </visual>
@@ -164,5 +164,5 @@
     <visual>
       <geometry>
-          <mesh filename="package://onigiri_war/models/tags/test.dae" scale="0.666 0.666 1.0"/>
+          <mesh filename="package://burger_war/models/tags/test.dae" scale="0.666 0.666 1.0"/>
       </geometry>
     </visual>
@@ -176,5 +176,5 @@
     <visual>
       <geometry>
-          <mesh filename="package://onigiri_war/models/tags/0051g.dae" scale="0.666 0.666 1.0" />
+          <mesh filename="package://burger_war/models/tags/0051g.dae" scale="0.666 0.666 1.0" />
       </geometry>
     </visual>
@@ -188,5 +188,5 @@
     <visual>
       <geometry>
-          <mesh filename="package://onigiri_war/models/tags/test.dae" scale="0.666 0.666 1.0"/>
+          <mesh filename="package://burger_war/models/tags/test.dae" scale="0.666 0.666 1.0"/>
       </geometry>
     </visual>
@@ -200,5 +200,5 @@
     <visual>
       <geometry>
-          <mesh filename="package://onigiri_war/models/tags/0052g.dae" scale="0.666 0.666 1.0" />
+          <mesh filename="package://burger_war/models/tags/0052g.dae" scale="0.666 0.666 1.0" />
       </geometry>
     </visual>
@@ -212,10 +212,10 @@
     <visual>
       <geometry>
-          <mesh filename="package://onigiri_war/models/tags/test.dae" scale="0.666 0.666 1.0"/>
+          <mesh filename="package://burger_war/models/tags/test.dae" scale="0.666 0.666 1.0"/>
       </geometry>
     </visual>
   </link>
   <joint name="poll_joint" type="fixed">
-    <origin rpy="0 0 0" xyz="-0.09 0.0 0.12"/>
+    <origin rpy="0 0 0" xyz="-0.09 0.0 0.15"/>
     <parent link="base_link"/>
     <child link="poll"/>
@@ -229,5 +229,5 @@
   </link>
   <joint name="ball_joint" type="fixed">
-    <origin rpy="0 0 0" xyz="-0.09 0.0 0.21"/>
+    <origin rpy="0 0 0" xyz="-0.09 0.0 0.3"/>
     <parent link="base_link"/>
     <child link="ball"/>
