Commit message: modify robot tag

File: burger_war/models/red_bot.urdf.xacro (robot description, xacro)
@@ -3,5 +3,5 @@
   <xacro:include filename="$(find turtlebot3_description)/urdf/common_properties.xacro"/>
   <!-- xacro:include filename="$(find turtlebot3_description)/urdf/turtlebot3_burger.gazebo.xacro"/-->
-  <xacro:include filename="$(find burger_war)/models/hoge.gazebo.xacro"/>
+  <xacro:include filename="$(find burger_war)/models/burgerbot.gazebo.xacro"/>
   <link name="base_footprint"/>
   <joint name="base_joint" type="fixed">
@@ -152,5 +152,5 @@
       <geometry>
           <!-- 120mm x 0.666 = 80mm -->
-          <mesh filename="package://burger_war/models/tags/0050g.dae" scale="0.666 0.666 1.0" />
+          <mesh filename="package://burger_war/models/tags/0040g.dae" scale="0.666 0.666 1.0" />
       </geometry>
     </visual>
@@ -176,5 +176,5 @@
     <visual>
       <geometry>
-          <mesh filename="package://burger_war/models/tags/0051g.dae" scale="0.666 0.666 1.0" />
+          <mesh filename="package://burger_war/models/tags/0041g.dae" scale="0.666 0.666 1.0" />
       </geometry>
     </visual>
@@ -200,5 +200,5 @@
     <visual>
       <geometry>
-          <mesh filename="package://burger_war/models/tags/0052g.dae" scale="0.666 0.666 1.0" />
+          <mesh filename="package://burger_war/models/tags/0042g.dae" scale="0.666 0.666 1.0" />
       </geometry>
     </visual>
