Commit message: modifi poll and ball size. add color plate. #23 #24

File: burger_war/models/burgerbot.gazebo.xacro (robot description, xacro)
@@ -162,5 +162,11 @@
   </gazebo>
   <gazebo reference="poll">
-    <material>Gazebo/DarkGrey</material>
+    <material>Gazebo/White</material>
+  </gazebo>
+  <gazebo reference="blue_plate">
+    <material>Gazebo/Blue</material>
+  </gazebo>
+  <gazebo reference="red_plate">
+    <material>Gazebo/Red</material>
   </gazebo>
 </robot>
